Commit message: second commit

File: src/husky/husky_description/urdf/husky.urdf.xacro (robot description, xacro)
@@ -51,5 +51,5 @@
   <xacro:property name="wheel_length" value="0.1143" />
   <xacro:property name="wheel_radius" value="0.1651" />
-  <link name="solarPanel_link">
+  <!--link name="solarPanel_link">
    <inertial>
      <origin xyz="0 0 0" rpy="0 0 0"/>
@@ -69,5 +69,5 @@
      <origin xyz="0 0 0" rpy="0 0 0"/>
      <geometry>
-       <box size="1.0 1.6 0.05" />
+       <box size="1.5 1.5 0.05" />
      </geometry>
    </collision>
@@ -84,14 +84,14 @@
        </contact>
    </surface>
-  </link>
-  <gazebo reference="solarPanel_link">
+  </link-->
+  <!--gazebo reference="solarPanel_link">
     <mu1 value="10"/>
     <mu2 value="10"/>
-  </gazebo>
-  <joint name="base_to_panel_joint" type="fixed">
+  </gazebo-->
+  <!--joint name="base_to_panel_joint" type="fixed">
     <origin xyz="0 0 0.2" rpy="0 0 0" />
     <parent link="base_link"/>
     <child link="solarPanel_link"/>
-  </joint>
+  </joint-->
   <!-- Base link is the center of the robot's bottom plate -->
   <link name="base_link">

Commit message: 1st changes

File: src/husky/husky_description/urdf/husky.urdf.xacro (robot description, xacro)
@@ -51,5 +51,5 @@
   <xacro:property name="wheel_length" value="0.1143" />
   <xacro:property name="wheel_radius" value="0.1651" />
-  <!--link name="solarPanel_link">
+  <link name="solarPanel_link">
    <inertial>
      <origin xyz="0 0 0" rpy="0 0 0"/>
@@ -84,14 +84,14 @@
        </contact>
    </surface>
-  </link-->
+  </link>
   <!--gazebo reference="solarPanel_link">
     <mu1 value="10"/>
     <mu2 value="10"/>
   </gazebo-->
-  <!--joint name="base_to_panel_joint" type="fixed">
+  <joint name="base_to_panel_joint" type="fixed">
     <origin xyz="0 0 0.2" rpy="0 0 0" />
     <parent link="base_link"/>
     <child link="solarPanel_link"/>
-  </joint-->
+  </joint>
   <!-- Base link is the center of the robot's bottom plate -->
   <link name="base_link">

Commit message: second changes

File: src/husky/husky_description/urdf/husky.urdf.xacro (robot description, xacro)
@@ -22,8 +22,14 @@
 -->
 <robot name="husky" xmlns:xacro="http://ros.org/wiki/xacro">
-  <xacro:arg name="laser_enabled" default="true" />
+  <xacro:arg name="laser_enabled" default="$(optenv HUSKY_LMS1XX_ENABLED 0)" />
   <xacro:arg name="laser_xyz" default="$(optenv HUSKY_LMS1XX_XYZ 0.2206 0.0 0.00635)" />
   <xacro:arg name="laser_rpy" default="$(optenv HUSKY_LMS1XX_RPY 0.0 0.0 0.0)" />
-  <xacro:arg name="realsense_enabled" default="false" />
+  <xacro:arg name="laser_secondary_enabled" default="$(optenv HUSKY_LMS1XX_SECONDARY_ENABLED 0)" />
+  <xacro:arg name="laser_secondary_xyz" default="$(optenv HUSKY_LMS1XX_SECONDARY_XYZ -0.2206 0.0 0.00635)" />
+  <xacro:arg name="laser_secondary_rpy" default="$(optenv HUSKY_LMS1XX_SECONDARY_RPY 0.0 0.0 3.14159)" />
+  <xacro:arg name="laser_3d_enabled" default="$(optenv HUSKY_LASER_3D_ENABLED 0)" />
+  <xacro:arg name="laser_3d_xyz" default="$(optenv HUSKY_LASER_3D_XYZ 0 0 0)" />
+  <xacro:arg name="laser_3d_rpy" default="$(optenv HUSKY_LASER_3D_RPY 0 0 0)" />
+  <xacro:arg name="realsense_enabled" default="$(optenv HUSKY_REALSENSE_ENABLED 0)" />
   <xacro:arg name="realsense_xyz" default="$(optenv HUSKY_REALSENSE_XYZ 0 0 0)" />
   <xacro:arg name="realsense_rpy" default="$(optenv HUSKY_REALSENSE_RPY 0 0 0)" />
@@ -31,4 +37,7 @@
   <xacro:property name="husky_front_bumper_extend" value="$(optenv HUSKY_FRONT_BUMPER_EXTEND 0)" />
   <xacro:property name="husky_rear_bumper_extend" value="$(optenv HUSKY_REAR_BUMPER_EXTEND 0)" />
+  <!-- Height of the sensor arch in mm.  Must be either 510 or 300 -->
+  <xacro:arg name="sensor_arch_height"  default="$(optenv HUSKY_SENSOR_ARCH_HEIGHT 510)" />
+  <xacro:arg name="sensor_arch"         default="$(optenv HUSKY_SENSOR_ARCH 0)" />
   <xacro:arg name="robot_namespace" default="/" />
   <xacro:arg name="urdf_extras" default="empty.urdf" />
@@ -39,4 +48,5 @@
   <xacro:include filename="$(find husky_description)/urdf/accessories/sick_lms1xx_mount.urdf.xacro"/>
   <xacro:include filename="$(find husky_description)/urdf/accessories/sensor_arch.urdf.xacro"/>
+  <xacro:include filename="$(find husky_description)/urdf/accessories/vlp16_mount.urdf.xacro"/>
   <xacro:property name="M_PI" value="3.14159"/>
   <!-- Base Size -->
@@ -85,8 +95,4 @@
    </surface>
   </link>
-  <!--gazebo reference="solarPanel_link">
-    <mu1 value="10"/>
-    <mu2 value="10"/>
-  </gazebo-->
   <joint name="base_to_panel_joint" type="fixed">
     <origin xyz="0 0 0.2" rpy="0 0 0" />
@@ -107,10 +113,10 @@
         <box size="${ base_x_size + husky_front_bumper_extend + husky_rear_bumper_extend } ${base_y_size} ${base_z_size/2}"/>
       </geometry>
-    </collision>/husky0/imu/data
+    </collision>
     <collision>
       <origin xyz="0 0 ${base_z_size*3/4-0.01}" rpy="0 0 0" />
       <geometry>
         <box size="${base_x_size*4/5} ${base_y_size} ${base_z_size/2-0.02}"/>
-      </geometry>/husky0/imu/data
+      </geometry>
     </collision>
   </link>
@@ -159,33 +165,54 @@
   </xacro:husky_wheel>
   <xacro:husky_decorate />
+  <!--
+    Add the primary and secondary lasers
+  -->
   <xacro:if value="$(arg laser_enabled)">
-    <sick_lms1xx_mount prefix="base"/>
-    <sick_lms1xx frame="base_laser" topic="scan" robot_namespace="$(arg robot_namespace)"/>
+    <xacro:sick_lms1xx_mount prefix="base"/>
+    <xacro:sick_lms1xx frame="base_laser" topic="scan" robot_namespace="$(arg robot_namespace)"/>
     <joint name="laser_mount_joint" type="fixed">
       <origin xyz="$(arg laser_xyz)" rpy="$(arg laser_rpy)" />
       <parent link="top_plate_link" />
-      <child link="base_laser_mount_3" />
+      <child link="base_laser_mount" />
     </joint>
   </xacro:if>
+  <xacro:if value="$(arg laser_secondary_enabled)">
+    <xacro:sick_lms1xx_mount prefix="rear"/>
+    <xacro:sick_lms1xx frame="rear_laser" topic="rear/scan" robot_namespace="$(arg robot_namespace)"/>
+    <joint name="laser_secondary_mount_joint" type="fixed">
+      <origin xyz="$(arg laser_secondary_xyz)" rpy="$(arg laser_secondary_rpy)" />
+      <parent link="top_plate_link" />
+      <child link="rear_laser_mount" />
+    </joint>
+  </xacro:if>
   <!--
-    top sensor arch; include this if we have realsense enabled
-    keep this as a property to make it easier to add multiple conditions, should we need
-    the top bar for any additional sensors in the future
+    Add the main sensor arch if the user has specifically enabled it, or if a sensor
+    requires it for mounting
   -->
-  <xacro:property name="topbar_needed_realsense" value="$(arg realsense_enabled)" />
-  <xacro:if value="${topbar_needed_realsense}">
-    <xacro:sensor_arch prefix="" parent="top_plate_link">
-      <origin xyz="-0.35 0 0.51" rpy="0 0 -3.14"/>
-    </xacro:sensor_arch>
-  </xacro:if>
-  <!-- add the intel realsense to the topbar if needed -->
+  <xacro:property name="sensorbar_user_enabled"     value="$(arg sensor_arch)" />
+  <xacro:property name="sensorbar_needed_realsense" value="$(arg realsense_enabled)" />
+  <xacro:property name="sensorbar_needed_lidar"     value="$(arg laser_3d_enabled)" />
+  <xacro:if value="${sensorbar_needed_realsense or sensorbar_user_enabled or sensorbar_needed_lidar}">
+    <xacro:sensor_arch prefix="" parent="top_plate_link" size="$(arg sensor_arch_height)">
+        <origin xyz="$(optenv HUSKY_SENSOR_ARCH_OFFSET 0 0 0)" rpy="$(optenv HUSKY_SENSOR_ARCH_RPY 0 0 0)"/>
+      </xacro:sensor_arch>
+  </xacro:if>
+  <!-- add the intel realsense to the sensor arch if needed -->
   <xacro:if value="$(arg realsense_enabled)">
     <link name="realsense_mountpoint"/>
     <joint name="realsense_mountpoint_joint" type="fixed">
-      <origin xyz="0 0 0" rpy="0 0 -3.14159" />
+      <origin xyz="$(arg realsense_xyz)" rpy="$(arg realsense_rpy)" />
       <parent link="$(arg realsense_mount)"/>
       <child link="realsense_mountpoint" />
     </joint>
     <xacro:intel_realsense_mount prefix="camera" topic="realsense" parent_link="realsense_mountpoint"/>
+  </xacro:if>
+  <!--
+    Add the 3d laser to the sensor arch if needed
+  -->
+  <xacro:if value="$(arg laser_3d_enabled)">
+    <xacro:vlp16_mount prefix="" parent_link="sensor_arch_mount_link" topic="$(optenv HUSKY_LASER_3D_TOPIC points)">
+      <origin xyz="$(arg laser_3d_xyz)" rpy="$(arg laser_3d_rpy)" />
+    </xacro:vlp16_mount>
   </xacro:if>
   <gazebo>
@@ -195,5 +222,5 @@
     </plugin>
   </gazebo>
-  <!--gazebo>
+  <gazebo>
     <plugin name="imu_controller" filename="libhector_gazebo_ros_imu.so">
       <robotNamespace>$(arg robot_namespace)</robotNamespace>
@@ -208,6 +235,6 @@
       <headingGaussianNoise>0.005</headingGaussianNoise>
     </plugin>
-  </gazebo-->
-  <!--gazebo>
+  </gazebo>
+  <gazebo>
     <plugin name="gps_controller" filename="libhector_gazebo_ros_gps.so">
       <robotNamespace>$(arg robot_namespace)</robotNamespace>
@@ -223,17 +250,4 @@
       <drift>0.0001 0.0001 0.0001</drift>
     </plugin>
-  </gazebo-->
-  <gazebo>
-  <plugin name="p3d_base_controller" filename="libgazebo_ros_p3d.so">
-      <robotNamespace>$(arg robot_namespace)</robotNamespace>
-      <alwaysOn>true</alwaysOn>
-      <updateRate>50.0</updateRate>
-      <bodyName>base_link</bodyName>
-      <topicName>ground_truth/state</topicName>
-      <gaussianNoise>0.01</gaussianNoise>
-      <frameName>world</frameName>
-      <xyzOffsets>0 0 0</xyzOffsets>
-      <rpyOffsets>0 0 0</rpyOffsets>
-    </plugin>
   </gazebo>
   <!-- Optional custom includes. -->
