Commit message: add .rosinstall, update urdf

File: test/urdf/husky.urdf.xacro (robot description, xacro)
@@ -104,10 +104,10 @@
         <box size="${ base_x_size + husky_front_bumper_extend + husky_rear_bumper_extend } ${base_y_size} ${base_z_size/2}"/>
       </geometry>
-    </collision>/husky0/imu/data
+    </collision>
     <collision>
       <origin xyz="0 0 ${base_z_size*3/4-0.01}" rpy="0 0 0" />
       <geometry>
         <box size="${base_x_size*4/5} ${base_y_size} ${base_z_size/2-0.02}"/>
-      </geometry>/husky0/imu/data
+      </geometry>
     </collision>
   </link>
